File: controller-v3/helmholtz-controller-v2.kicad_pcb (KiCad board)
At the start: 2 copper layers, 72.7 x 72.1 mm, 60 parts, among them J1 Screw_Terminal_01x02, J2 Screw_Terminal_01x02, J3 Screw_Terminal_01x02, J4 Screw_Terminal_01x02, J5 Conn_01x04, U1 BDS63150AFM, U2 BDS63150AFM, U3 INA226, U4 INA226, U5 BDS63150AFM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

Commit message: Board mostly laid out
Parts:
- removed R12: 6.8k, Resistor_SMD:R_0603_1608Metric
- removed R13: 100m, Resistor_SMD:R_1206_3216Metric
- removed R14: 10k, Resistor_SMD:R_0603_1608Metric
- J1, J2, J3: footprint TerminalBlock_Phoenix:TerminalBlock_Phoenix_PT-1,5-2-3.5-H_1x02_P3.50mm_Horizontal -> Connector_AMASS:AMASS_XT30PW-F_1x02_P2.50mm_Horizontal
- R1, R9: value 10k -> R_US
- R11, R4, R6: value 30k -> R_US
- R2, R8: value 100m -> R_US; footprint Resistor_SMD:R_1206_3216Metric -> Resistor_SMD:R_0603_1608Metric
- R3, R7: value 6.8k -> R_US
- U1, U2, U5: value BDS63150AFM -> DRV8871DDA; footprint psas-footprints:U-BD63150AFM -> Package_SO:Texas_HTSOP-8-1EP_3.9x4.9mm_P1.27mm_EP2.95x4.9mm_Mask2.4x3.1mm_ThermalVias
- moved R2 44.5 mm to (214.8, 140.3), turned to 180 degrees
- moved R7 33.5 mm to (225.8, 95.2), turned to 0 degrees
- moved R11 31.4 mm to (221.2, 114.8), turned to 90 degrees
- moved C3 28.1 mm to (211.4, 115.6), turned to 180 degrees
- moved U2 24.2 mm to (213.0, 144.1), turned to 180 degrees
- moved R8 23.4 mm to (220.2, 139.1), turned to 90 degrees
- moved C2 21.5 mm to (211.5, 140.3), turned to 180 degrees
- moved U5 20.0 mm to (212.9, 119.5), turned to 180 degrees
- moved TP4 18.7 mm to (224.1, 117.6)
- moved R6 17.9 mm to (222.8, 144.8), turned to -90 degrees
- moved TP5 17.3 mm to (225.0, 96.7)
- moved TP6 17.1 mm to (224.8, 101.4)
- moved R9 15.6 mm to (224.1, 120.5), turned to -90 degrees
- moved C1 13.7 mm to (211.1, 95.8), turned to 180 degrees
- moved TP1 13.5 mm to (222.8, 141.3)
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Connections:
- net /D6 renamed Net-(U7-GPIO13)
- J5 pad 1: +3.3V -> unconnected-(J5-Pin_1-Pad1)
- R1 pad 1: +3.3V -> Net-(U1-ILIM)
- R1 pad 2: /X_FAIL -> GND
- R10 pad 2: Net-(J2-Pin_1) -> Net-(J2-Pin_2)
- R11 pad 1: +3.3V -> /Y_IN1
- R11 pad 2: Net-(U5-VREF) -> GND
- R15 pad 1: Net-(U6-Vbus) -> Net-(U2-OUT1)
- R15 pad 2: Net-(J3-Pin_1) -> Net-(J3-Pin_2)
- R2 pad 1: Net-(U1-RNFS) -> Net-(U2-ILIM)
- R3 pad 1: GND -> Net-(U5-ILIM)
- R3 pad 2: Net-(U1-VREF) -> GND
- R4 pad 1: +3.3V -> /X_IN2
- R4 pad 2: Net-(U1-VREF) -> GND
- R5 pad 1: Net-(U4-Vbus) -> Net-(U1-OUT1)
- R5 pad 2: Net-(J1-Pin_1) -> Net-(J1-Pin_2)
- R6 pad 1: +3.3V -> /Z_IN2
- R6 pad 2: Net-(U2-VREF) -> GND
- R7 pad 1: GND -> /X_IN1
- R7 pad 2: Net-(U2-VREF) -> GND
- R8 pad 1: Net-(U2-RNFS) -> /Z_IN1
- R9 pad 1: /Y_FAIL -> /Y_IN2
- R9 pad 2: +3.3V -> GND
- U1 pad 1: Net-(U4-Vbus) -> GND
- U1 pad 2: Net-(U4-Vbus) -> /X_IN2
- U1 pad 3: Net-(U4-Vbus) -> /X_IN1
- U1 pad 4: unconnected-(U1-NC-Pad4) -> Net-(U1-ILIM)
- U1 pad 5: unconnected-(U1-NC-Pad5) -> +12V
- U1 pad 6: Net-(J1-Pin_2) -> Net-(U1-OUT1)
- U1 pad 7: Net-(J1-Pin_2) -> GND
- U1 pad 8: Net-(J1-Pin_2) -> Net-(J1-Pin_1)
- U1 pad 9: unconnected-(U1-NC-Pad9) -> GND
- U2 pad 1: Net-(U3-Vbus) -> GND
- U2 pad 2: Net-(U3-Vbus) -> /Z_IN2
- U2 pad 3: Net-(U3-Vbus) -> /Z_IN1
- U2 pad 4: unconnected-(U2-NC-Pad4) -> Net-(U2-ILIM)
- U2 pad 5: unconnected-(U2-NC-Pad5) -> +12V
- U2 pad 6: Net-(J2-Pin_2) -> Net-(U2-OUT1)
- U2 pad 7: Net-(J2-Pin_2) -> GND
- U2 pad 8: Net-(J2-Pin_2) -> Net-(J3-Pin_1)
- U2 pad 9: unconnected-(U2-NC-Pad9) -> GND
- U3 pad 9: Net-(J2-Pin_1) -> Net-(J2-Pin_2)
- U4 pad 10: Net-(U4-Vbus) -> Net-(U1-OUT1)
- U4 pad 8: Net-(U4-Vbus) -> Net-(U1-OUT1)
- U4 pad 9: Net-(J1-Pin_1) -> Net-(J1-Pin_2)
- U5 pad 1: Net-(U6-Vbus) -> GND
- U5 pad 2: Net-(U6-Vbus) -> /Y_IN2
- U5 pad 3: Net-(U6-Vbus) -> /Y_IN1
- U5 pad 4: unconnected-(U5-NC-Pad4) -> Net-(U5-ILIM)
- U5 pad 5: unconnected-(U5-NC-Pad5) -> +12V
- U5 pad 6: Net-(J3-Pin_2) -> Net-(U3-Vbus)
- U5 pad 7: Net-(J3-Pin_2) -> GND
- U5 pad 8: Net-(J3-Pin_2) -> Net-(J2-Pin_1)
- U5 pad 9: unconnected-(U5-NC-Pad9) -> GND
- U6 pad 10: Net-(U6-Vbus) -> Net-(U2-OUT1)
- U6 pad 8: Net-(U6-Vbus) -> Net-(U2-OUT1)
- U6 pad 9: Net-(J3-Pin_1) -> Net-(J3-Pin_2)
- U7 pad 11: /Y_FAIL -> unconnected-(U7-GPIO8-Pad11)
- U7 pad 16: /Z_FAIL -> /Z_INA_ALERT
- U7 pad 29: /Z_INA_ALERT -> unconnected-(U7-GPIO22-Pad29)
- U7 pad 6: /X_FAIL -> unconnected-(U7-GPIO4-Pad6)
Routing:
- net +3.3V: track 248.3 -> 82.4 mm, vias 0 -> 15
- net GND: track 55.9 -> 1.32 mm, vias 178 -> 107
- net /Z_FAIL: track 38.1 -> 0.00 mm, vias 2 -> 0
- net /Y_FAIL: track 31.6 -> 0.00 mm, vias 2 -> 0
- net /X_FAIL: track 26.2 -> 0.00 mm, vias 2 -> 0
- net /Z_INA_ALERT: track 57.8 -> 32.4 mm
- net /Y_IN2: track 37.4 -> 21.7 mm, vias 2 -> 0
- net Net-(U2-OUT1): track 0.00 -> 15.4 mm
- net Net-(U1-OUT1): track 0.00 -> 15.1 mm
- net Net-(J3-Pin_2): track 0.00 -> 14.5 mm
- net Net-(J1-Pin_2): track 0.00 -> 14.1 mm
- net Net-(J2-Pin_2): track 0.25 -> 13.4 mm
- net /Y_IN1: track 34.9 -> 22.2 mm, vias 2 -> 0
- net /X_IN2: track 30.4 -> 19.5 mm, vias 1 -> 0
- net /X_IN1: track 29.7 -> 19.2 mm, vias 1 -> 0
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- added copper zone on B.Cu, net +12V
- added copper zone on B.Cu, net +3.3V
- added copper zone on F.Cu, net +3.3V
- removed copper zone on F.Cu, net Net-(J1-Pin_2)
- removed copper zone on F.Cu, net Net-(J2-Pin_2)
- removed copper zone on F.Cu, net Net-(J3-Pin_2)
- removed copper zone on F.Cu, net Net-(U1-RNFS)
- removed copper zone on F.Cu, net Net-(U2-RNFS)
- removed copper zone on F.Cu, net Net-(U3-Vbus)
- removed copper zone on F.Cu, net Net-(U4-Vbus)
- removed copper zone on F.Cu, net Net-(U5-RNFS)
- removed copper zone on F.Cu, net Net-(U6-Vbus)

Commit message: getting closer to perfect
Parts:
- moved C5 0.39 mm to (208.7, 113.3)
- moved C7 0.28 mm to (210.1, 135.9)
- moved C6 0.20 mm to (209.5, 92.5)
Routing:
- net +12V: track 62.0 -> 5.25 mm
- net +3.3V: track 82.4 -> 84.0 mm, vias 15 -> 11
- net /Y_INA_ALERT: track 37.5 -> 38.3 mm
- net GND: vias 107 -> 135
Other:
- board text added: "+"
