File: controller-v3/helmholtz-controller-v2.kicad_pcb (KiCad board)
At the start: 2 copper layers, 72.7 x 72.1 mm, 57 parts, among them J1 Screw_Terminal_01x02, J2 Screw_Terminal_01x02, J3 Screw_Terminal_01x02, J4 Screw_Terminal_01x02, J5 Conn_01x04, U1 DRV8871DDA, U2 DRV8871DDA, U3 INA226, U4 INA226, U5 DRV8871DDA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

Commit message: Done!
Parts:
- R1, R3: value R_US -> 32k
- R11, R4, R6, R7, R8, R9: value R_US -> 10k
- R2: value R_US -> 32K
- moved R16 0.72 mm to (228.5, 92.2)
- moved R17 0.72 mm to (228.5, 90.8)
- moved TP7 0.27 mm to (226.1, 92.2)
- moved R20 0.26 mm to (234.1, 142.6)
- moved D4 0.13 mm to (234.1, 145.6)
Routing:
- net +3.3V: track 84.0 -> 83.0 mm
Other:
- board text added: "Helmholtz Controller Board 3.0 2026-3-22"
- board text removed: "Helmholtz Controller Board ${REVISION} ${ISSUE_DATE}"

Commit message: Some polish
Parts:
- moved TP10 1.69 mm to (257.2, 98.5)
- moved C3 0.10 mm to (211.4, 115.7)
Routing:
- net +3.3V: track 83.0 -> 81.4 mm
- net GND: vias 135 -> 141
Changed lines of the file:
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@@
 			(at 0 1.83 180)
 			(layer "F.Fab")
+			(hide yes)
 			(effects
 				(font
@@
 			(layer "F.Fab")
 		)
-		(fp_text user "${REFERENCE}"
-			(at 0 0 180)
-			(layer "F.Fab")
-			(effects
-				(font
-					(size 0.8 0.8)
-					(thickness 0.12)
-				)
-			)
-		)
 		(pad "1" smd roundrect
 			(at -1.4625 0 180)
@@
 	(footprint "oresat-misc:TestPoint-0.75mm-th"
 		(layer "F.Cu")
-		(at 258.29 97.17)
+		(at 257.25 98.5)
 		(property "Reference" "TP10"
 			(at 0.66 -1.52 0)
@@
 			(at 0 2.45 0)
 			(layer "F.Fab")
+			(hide yes)
 			(effects
 				(font
@@
 	(footprint "Capacitor_SMD:C_0805_2012Metric"
 		(layer "F.Cu")
-		(at 211.4 115.6 180)
+		(at 211.4 115.7 180)
 		(descr "Capacitor SMD 0805 (2012 Metric), square (rectangular) end terminal, IPC-7351 nominal, (Body size source: IPC-SM-782 page 76, https://www.pcb-3d.com/wordpress/wp-content/uploads/ipc-sm-782a_amendment_1_and_2.pdf, https://docs.google.com/spreadsheets/d/1BsfQQcO9C6DZCsRaXUlFlo91Tg2WpOkGARC1WS5S8t0/edit?usp=sharing), generated with kicad-footprint-generator")
 		(tags "capacitor")
@@
 	)
 	(segment
+		(start 229.3 90.1)
+		(end 228.4 89.2)
+		(width 0.2)
+		(layer "F.Cu")
+		(net 3)
+	)
+	(segment
 		(start 201.82 136.26)
 		(end 202.16 136.6)
@@
 	)
 	(segment
-		(start 229.3 90.75)
-		(end 227.75 89.2)
+		(start 232.1849 89.545)
+		(end 229.855 89.545)
 		(width 0.2)
 		(layer "F.Cu")
@@
 	)
 	(segment
-		(start 227.75 89.2)
-		(end 226.1 89.2)
+		(start 229.3 90.75)
+		(end 229.3 90.1)
 		(width 0.2)
 		(layer "F.Cu")
@@
 	)
 	(segment
-		(start 202.16 136.6)
-		(end 203.3 136.6)
-		(width 0.1524)
+		(start 229.855 89.545)
+		(end 229.3 90.1)
+		(width 0.2)
 		(layer "F.Cu")
 		(net 3)
 	)
 	(segment
-		(start 230.505 89.545)
-		(end 229.3 90.75)
-		(width 0.2)
+		(start 202.16 136.6)
+		(end 203.3 136.6)
+		(width 0.1524)
 		(layer "F.Cu")
 		(net 3)
@@
 	)
 	(segment
-		(start 232.1849 89.545)
-		(end 230.505 89.545)
-		(width 0.2)
-		(layer "F.Cu")
-		(net 3)
-	)
-	(segment
 		(start 200.57 113.72)
 		(end 201.82 113.72)
@@
 	)
 	(segment
+		(start 228.4 89.2)
+		(end 226.1 89.2)
+		(width 0.2)
+		(layer "F.Cu")
+		(net 3)
+	)
+	(segment
 		(start 202.155 135.595)
 		(end 201.82 135.93)
@@
 	)
 	(segment
+		(start 257.25 98.5)
+		(end 257.25 100.755)
+		(width 0.1524)
+		(layer "F.Cu")
+		(net 4)
+	)
+	(segment
 		(start 203.3 112.7)
 		(end 204.85 111.15)
@@
 	)
 	(segment
-		(start 251.5651 99.705)
-		(end 256.2 99.705)
-		(width 1)
+		(start 257.25 100.755)
+		(end 257.355 100.86)
+		(width 0.1524)
 		(layer "F.Cu")
 		(net 4)
@@
 	)
 	(segment
+		(start 257.355 100.86)
+		(end 256.41 100.86)
+		(width 0.2)
+		(layer "F.Cu")
+		(net 4)
+	)
+	(segment
 		(start 210.55 113.85)
 		(end 210.4 114)
@@
 	)
 	(segment
+		(start 256.41 100.86)
+		(end 255.255 99.705)
+		(width 0.2)
+		(layer "F.Cu")
+		(net 4)
+	)
+	(segment
+		(start 255.255 99.705)
+		(end 251.5651 99.705)
+		(width 0.2)
+		(layer "F.Cu")
+		(net 4)
+	)
+	(segment
 		(start 210.55 111.6)
 		(end 210.55 113.85)
@@
 	)
 	(segment
-		(start 258.29 97.17)
-		(end 257.823 97.17)
-		(width 0.2)
-		(layer "F.Cu")
-		(net 4)
-	)
-	(segment
-		(start 256.2 99.705)
-		(end 257.355 100.86)
-		(width 1)
-		(layer "F.Cu")
-		(net 4)
-	)
-	(segment
 		(start 201.8 112.7)
 		(end 203.3 112.7)
@@
 	)
 	(segment
-		(start 257.823 97.17)
-		(end 255.319 99.674)
-		(width 0.2)
-		(layer "F.Cu")
-		(net 4)
-	)
-	(segment
 		(start 209.25 93.7)
 		(end 209.3 93.65)
@@
 	)
 	(segment
-		(start 226.125 92.25)
-		(end 226.125 92.675)
-		(width 0.2)
-		(layer "F.Cu")
-		(net 6)
-	)
-	(segment
 		(start 226.35 92.5)
 		(end 226.3 92.45)
@@
 	)
 	(segment
-		(start 228.1 93.45)
-		(end 229.3 92.25)
+		(start 200.12 114.22)
+		(end 201.82 114.22)
 		(width 0.2)
 		(layer "F.Cu")
@@
 	)
 	(segment
-		(start 200.12 114.22)
-		(end 201.82 114.22)
+		(start 228.5 93.45)
+		(end 229.3 92.65)
 		(width 0.2)
 		(layer "F.Cu")
@@
 	)
 	(segment
-		(start 226.9 93.45)
-		(end 228.1 93.45)
+		(start 226.125 92.25)
+		(end 226.125 92.675)
 		(width 0.2)
 		(layer "F.Cu")
@@
 	)
 	(segment
-		(start 199.65 93.65)
-		(end 199.65 91.7)
+		(start 229.3 92.65)
+		(end 229.3 92.25)
 		(width 0.2)
 		(layer "F.Cu")
@@
 	)
 	(segment
-		(start 200.1 136.45)
-		(end 200.75 137.1)
+		(start 199.65 93.65)
+		(end 199.65 91.7)
 		(width 0.2)
 		(layer "F.Cu")
@@
 		(net 6)
 	)
+	(segment
+		(start 226.9 93.45)
+		(end 228.5 93.45)
+		(width 0.2)
+		(layer "F.Cu")
+		(net 6)
+	)
+	(segment
+		(start 200.1 136.45)
+		(end 200.75 137.1)
+		(width 0.2)
+		(layer "F.Cu")
+		(net 6)
+	)
 	(via
 		(at 199.65 93.65)
@@
 	)
 	(via
+		(at 220.15 137.4)
+		(size 0.508)
+		(drill 0.254)
+		(layers "F.Cu" "B.Cu")
+		(free yes)
+		(net 7)
+	)
+	(via
 		(at 229.825 107.525)
 		(size 0.508)
@@
 	)
 	(via
+		(at 215.65 122.6)
+		(size 0.508)
+		(drill 0.254)
+		(layers "F.Cu" "B.Cu")
+		(free yes)
+		(net 7)
+	)
+	(via
 		(at 245.5 157.7)
 		(size 0.508)
@@
 	)
 	(via
+		(at 222.8 146.4)
+		(size 0.508)
+		(drill 0.254)
+		(layers "F.Cu" "B.Cu")
+		(free yes)
+		(net 7)
+	)
+	(via
 		(at 221.15 92.4)
 		(size 0.508)
@@
 	)
 	(via
+		(at 215.5 147.35)
+		(size 0.508)
+		(drill 0.254)
+		(layers "F.Cu" "B.Cu")
+		(free yes)
+		(net 7)
+	)
+	(via
 		(at 260.6 120)
 		(size 0.508)
@@
 	)
 	(via
-		(at 210.45 125.65)
+		(at 208.425 92.375)
 		(size 0.508)
 		(drill 0.254)
@@
 	)
 	(via
-		(at 208.425 92.375)
+		(at 212.35 114.45)
 		(size 0.508)
 		(drill 0.254)
@@
 	)
 	(via
-		(at 260.5 157.6)
+		(at 208.4 120.1)
 		(size 0.508)
 		(drill 0.254)
@@
 	)
 	(via
-		(at 257.675 142.85)
+		(at 260.5 157.6)
 		(size 0.508)
 		(drill 0.254)
@@
 	)
 	(via
-		(at 203.7 142.6)
+		(at 257.675 142.85)
 		(size 0.508)
 		(drill 0.254)
@@
 	)
 	(via
-		(at 252.4 147.1)
+		(at 203.7 142.6)
 		(size 0.508)
 		(drill 0.254)
@@
 	)
 	(via
-		(at 260.6 140.5)
+		(at 252.4 147.1)
 		(size 0.508)
 		(drill 0.254)
@@
 	)
 	(via
-		(at 208.75 124.65)
+		(at 260.6 140.5)
 		(size 0.508)
 		(drill 0.254)
@@
 	)
 	(via
-		(at 221.8 112.05)
+		(at 221.2 113.2)
 		(size 0.508)
 		(drill 0.254)
@@
 	)
 	(via
+		(at 227.45 95.2)
+		(size 0.508)
+		(drill 0.254)
+		(layers "F.Cu" "B.Cu")
+		(free yes)
+		(net 7)
+	)
+	(via
 		(at 201.8 87.1)
 		(size 0.508)
@@
 	)
 	(via
+		(at 224.85 105.5)
+		(size 0.508)
+		(drill 0.254)
+		(layers "F.Cu" "B.Cu")
+		(free yes)
+		(net 7)
+	)
+	(via
 		(at 225.8 99)
 		(size 0.508)
@@
 		(polygon
 			(pts
-				(xy 208.6 115.15) (xy 211.3 115.15) (xy 211.3 117.65) (xy 208.3 117.65) (xy 208.3 115.15)
+				(xy 211.15 114.95) (xy 211.15 117.65) (xy 208.3 117.65) (xy 208.3 114.95)
 			)
 		)

Commit message: Requested changes
Parts:
- moved R15 0.90 mm to (205.5, 140.0)
- moved U6 0.90 mm to (205.5, 137.0)
- moved C7 0.90 mm to (210.1, 136.8)
Routing:
- net Net-(U2-OUT1): track 15.4 -> 14.4 mm
- net SCL: track 89.3 -> 90.3 mm
- net SDA: track 88.5 -> 89.4 mm
- net Net-(J2-Pin_2): track 13.4 -> 14.0 mm
- net GND: vias 141 -> 144
Other:
- board text added: "Shaelin Olton Jacob Lutz"
- board text removed: "Shaelin Olton"

Commit message: Latest push
Parts:
- moved R16 4.29 mm to (224.2, 91.5), turned to 90 degrees
- moved D6 4.29 mm to (242.0, 143.2), turned to 0 degrees
- moved R22 3.56 mm to (242.0, 141.6)
- moved D5 3.37 mm to (237.5, 143.2), turned to 0 degrees
- moved R4 2.64 mm to (224.2, 101.4), turned to 180 degrees
- moved D4 2.62 mm to (233.0, 143.2), turned to 0 degrees
- moved R21 2.42 mm to (237.5, 141.6)
- moved TP8 2.37 mm to (227.8, 90.8)
- moved TP6 1.71 mm to (225.0, 99.7)
- moved TP7 1.68 mm to (227.8, 92.4)
- moved R7 1.66 mm to (224.2, 95.3), turned to 180 degrees
- moved R20 1.45 mm to (233.0, 141.6)
- moved D2 1.44 mm to (258.2, 101.3)
- moved R17 1.19 mm to (229.3, 90.0), turned to 90 degrees
- moved R18 1.15 mm to (258.2, 99.7)
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Routing:
- net Net-(U7-GPIO13): track 24.3 -> 18.1 mm
- net +3.3V: track 81.4 -> 76.9 mm
- net Net-(U7-VBUS): track 18.7 -> 14.5 mm
- net Net-(D5-A): track 3.69 -> 0.00 mm
- net Net-(D6-A): track 3.69 -> 0.00 mm
- net SCL: track 90.3 -> 93.1 mm
- net Net-(D4-A): track 3.75 -> 1.57 mm
- net /X_INA_ALERT: track 46.7 -> 44.9 mm
- net /D5: track 12.2 -> 10.4 mm
- net /D4: track 5.23 -> 3.80 mm
- net /X_IN2: track 19.5 -> 18.5 mm
- net SDA: track 89.4 -> 90.0 mm
